File: ElectronBoardMKI.sch (EAGLE design)
At the start: 46 parts, among them IC1 7805TV, Q1 TN0602N3, Q2 TN0602N3, T2 2N2222, T3 2N2222, T4 2N2222, U1 LM386N

Commit message: Updated Parts
Parts:
- added RX_______TX: (no value), SparkFun-Connectors:CONN_02LOCK_LONGPADS
- C3: value 250uf -> 220uf
- C8: value 0.05uf -> 0.047uf; device resistor:CPOL-USE5-8.5 -> resistor:C-US050-035X075
- Q1, Q2: value TN0602N3 -> BSS170; device transistor-fet:TN0602N3 -> transistor-fet:BSS101
- renumbered SCL__SDA1 to SCL___SDA1, SCL__SDA2 to SCL___SDA2
Connections:
- new net RX: RX_______TX.1, U$1.RX
- new net TX: RX_______TX.2, U$1.TX
- net N$6: now also C8.1; no longer C8.+
- net N$7: now also C8.2; no longer C8.-
Changed lines of the file:
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@@
 <part name="GND6" library="supply1" library_urn="urn:adsk.eagle:library:371" deviceset="GND" device=""/>
 <part name="GND9" library="supply1" library_urn="urn:adsk.eagle:library:371" deviceset="GND" device=""/>
-<part name="SCL__SDA1" library="SparkFun-Connectors" library_urn="urn:adsk.eagle:library:513" deviceset="CONN_02" device="LOCK_LONGPADS" package3d_urn="urn:adsk.eagle:package:38047/1"/>
-<part name="SCL__SDA2" library="SparkFun-Connectors" library_urn="urn:adsk.eagle:library:513" deviceset="CONN_02" device="LOCK_LONGPADS" package3d_urn="urn:adsk.eagle:package:38047/1"/>
+<part name="SCL___SDA1" library="SparkFun-Connectors" library_urn="urn:adsk.eagle:library:513" deviceset="CONN_02" device="LOCK_LONGPADS" package3d_urn="urn:adsk.eagle:package:38047/1"/>
+<part name="SCL___SDA2" library="SparkFun-Connectors" library_urn="urn:adsk.eagle:library:513" deviceset="CONN_02" device="LOCK_LONGPADS" package3d_urn="urn:adsk.eagle:package:38047/1"/>
 <part name="IN-TEMP" library="SparkFun-Connectors" library_urn="urn:adsk.eagle:library:513" deviceset="CONN_03" device="LOCK_LONGPADS" package3d_urn="urn:adsk.eagle:package:38065/1"/>
 <part name="OUT-TEMP" library="SparkFun-Connectors" library_urn="urn:adsk.eagle:library:513" deviceset="CONN_03" device="LOCK_LONGPADS" package3d_urn="urn:adsk.eagle:package:38065/1"/>
@@
 <part name="C1" library="resistor" library_urn="urn:adsk.eagle:library:348" deviceset="CPOL-US" device="E5-8.5" package3d_urn="urn:adsk.eagle:package:25860/1" value="10uf"/>
 <part name="C2" library="resistor" library_urn="urn:adsk.eagle:library:348" deviceset="CPOL-US" device="E5-8.5" package3d_urn="urn:adsk.eagle:package:25860/1" value="1uf"/>
-<part name="Q1" library="transistor-fet" library_urn="urn:adsk.eagle:library:396" deviceset="TN0602N3" device="" package3d_urn="urn:adsk.eagle:package:28535/2"/>
+<part name="Q1" library="transistor-fet" library_urn="urn:adsk.eagle:library:396" deviceset="BSS101" device="" package3d_urn="urn:adsk.eagle:package:28523/2" value="BSS170"/>
 <part name="R12" library="resistor" library_urn="urn:adsk.eagle:library:348" deviceset="R-US_" device="0207/12" package3d_urn="urn:adsk.eagle:package:25938/1" value="4.7k"/>
 <part name="R13" library="resistor" library_urn="urn:adsk.eagle:library:348" deviceset="R-US_" device="0207/12" package3d_urn="urn:adsk.eagle:package:25938/1" value="4.7k"/>
-<part name="Q2" library="transistor-fet" library_urn="urn:adsk.eagle:library:396" deviceset="TN0602N3" device="" package3d_urn="urn:adsk.eagle:package:28535/2"/>
+<part name="Q2" library="transistor-fet" library_urn="urn:adsk.eagle:library:396" deviceset="BSS101" device="" package3d_urn="urn:adsk.eagle:package:28523/2" value="BSS170"/>
 <part name="R14" library="resistor" library_urn="urn:adsk.eagle:library:348" deviceset="R-US_" device="0207/12" package3d_urn="urn:adsk.eagle:package:25938/1" value="4.7k"/>
 <part name="R15" library="resistor" library_urn="urn:adsk.eagle:library:348" deviceset="R-US_" device="0207/12" package3d_urn="urn:adsk.eagle:package:25938/1" value="4.7k"/>
@@
 <part name="U1" library="SparkFun-IC-Amplifiers" library_urn="urn:adsk.eagle:library:520" deviceset="LM386" device="" package3d_urn="urn:adsk.eagle:package:38666/1" value="LM386N"/>
 <part name="C7" library="resistor" library_urn="urn:adsk.eagle:library:348" deviceset="CPOL-US" device="E5-8.5" package3d_urn="urn:adsk.eagle:package:25860/1" value="10uf"/>
-<part name="C8" library="resistor" library_urn="urn:adsk.eagle:library:348" deviceset="CPOL-US" device="E5-8.5" package3d_urn="urn:adsk.eagle:package:25860/1" value="0.05uf"/>
+<part name="C8" library="resistor" library_urn="urn:adsk.eagle:library:348" deviceset="C-US" device="050-035X075" package3d_urn="urn:adsk.eagle:package:26193/1" value="0.047uf"/>
 <part name="C9" library="resistor" library_urn="urn:adsk.eagle:library:348" deviceset="CPOL-US" device="E5-8.5" package3d_urn="urn:adsk.eagle:package:25860/1" value="1uf"/>
 <part name="R19" library="resistor" library_urn="urn:adsk.eagle:library:348" deviceset="R-US_" device="0207/12" package3d_urn="urn:adsk.eagle:package:25938/1" value="10k"/>
-<part name="C3" library="resistor" library_urn="urn:adsk.eagle:library:348" deviceset="CPOL-US" device="E5-8.5" package3d_urn="urn:adsk.eagle:package:25860/1" value="250uf"/>
+<part name="C3" library="resistor" library_urn="urn:adsk.eagle:library:348" deviceset="CPOL-US" device="E5-8.5" package3d_urn="urn:adsk.eagle:package:25860/1" value="220uf"/>
+<part name="RX_______TX" library="SparkFun-Connectors" library_urn="urn:adsk.eagle:library:513" deviceset="CONN_02" device="LOCK_LONGPADS" package3d_urn="urn:adsk.eagle:package:38047/1"/>
 </parts>
 <sheets>
@@
 <instance part="GND6" gate="1" x="-101.6" y="-86.36"/>
 <instance part="GND9" gate="1" x="-101.6" y="-104.14"/>
-<instance part="SCL__SDA1" gate="G$1" x="-58.42" y="88.9"/>
-<instance part="SCL__SDA2" gate="G$1" x="-58.42" y="71.12"/>
+<instance part="SCL___SDA1" gate="G$1" x="-58.42" y="88.9"/>
+<instance part="SCL___SDA2" gate="G$1" x="-58.42" y="71.12"/>
 <instance part="IN-TEMP" gate="J$1" x="-15.24" y="109.22"/>
 <instance part="OUT-TEMP" gate="J$1" x="-15.24" y="86.36"/>
@@
 <instance part="R19" gate="G$1" x="121.92" y="-17.78" rot="R90"/>
 <instance part="C3" gate="G$1" x="132.08" y="2.54" rot="R90"/>
+<instance part="RX_______TX" gate="G$1" x="-170.18" y="76.2"/>
 </instances>
 <busses>
@@
 <net name="SCL-5V" class="0">
 <segment>
-<pinref part="SCL__SDA1" gate="G$1" pin="2"/>
+<pinref part="SCL___SDA1" gate="G$1" pin="2"/>
 <wire x1="-50.8" y1="91.44" x2="-48.26" y2="91.44" width="0.1524" layer="91"/>
 <label x="-48.26" y="91.44" size="1.778" layer="95"/>
 </segment>
 <segment>
-<pinref part="SCL__SDA2" gate="G$1" pin="2"/>
+<pinref part="SCL___SDA2" gate="G$1" pin="2"/>
 <wire x1="-50.8" y1="73.66" x2="-48.26" y2="73.66" width="0.1524" layer="91"/>
 <label x="-48.26" y="73.66" size="1.778" layer="95"/>
@@
 <net name="SDA-5V" class="0">
 <segment>
-<pinref part="SCL__SDA1" gate="G$1" pin="1"/>
+<pinref part="SCL___SDA1" gate="G$1" pin="1"/>
 <wire x1="-50.8" y1="88.9" x2="-48.26" y2="88.9" width="0.1524" layer="91"/>
 <label x="-48.26" y="88.9" size="1.778" layer="95"/>
 </segment>
 <segment>
-<pinref part="SCL__SDA2" gate="G$1" pin="1"/>
+<pinref part="SCL___SDA2" gate="G$1" pin="1"/>
 <wire x1="-50.8" y1="71.12" x2="-48.26" y2="71.12" width="0.1524" layer="91"/>
 <label x="-48.26" y="71.12" size="1.778" layer="95"/>
@@
 <junction x="121.92" y="2.54"/>
 <pinref part="U1" gate="G1" pin="OUT"/>
-<pinref part="C8" gate="G$1" pin="+"/>
+<pinref part="C8" gate="G$1" pin="1"/>
 <pinref part="C3" gate="G$1" pin="+"/>
 </segment>
@@
 <wire x1="121.92" y1="-10.16" x2="121.92" y2="-12.7" width="0.1524" layer="91"/>
 <pinref part="R19" gate="G$1" pin="2"/>
-<pinref part="C8" gate="G$1" pin="-"/>
+<pinref part="C8" gate="G$1" pin="2"/>
 </segment>
 </net>
@@
 </segment>
 </net>
+<net name="RX" class="0">
+<segment>
+<pinref part="RX_______TX" gate="G$1" pin="1"/>
+<pinref part="U$1" gate="G$1" pin="RX"/>
+<wire x1="-162.56" y1="76.2" x2="-134.62" y2="76.2" width="0.1524" layer="91"/>
+</segment>
+</net>
+<net name="TX" class="0">
+<segment>
+<pinref part="U$1" gate="G$1" pin="TX"/>
+<pinref part="RX_______TX" gate="G$1" pin="2"/>
+<wire x1="-134.62" y1="81.28" x2="-134.62" y2="78.74" width="0.1524" layer="91"/>
+<wire x1="-134.62" y1="78.74" x2="-162.56" y2="78.74" width="0.1524" layer="91"/>
+</segment>
+</net>

Commit message: Display Board. Attained old board files. Schematic organization.
Parts:
- added C4, C5: 1uf, capacitor-wima:C2.5/4
- added SCREEN1: (no value), SparkFun-Connectors:CONN_05X2SHD
- added U4: NHD‐C0220, GEMS:NHD‐C0220
Connections:
- new net N$21: C4.2, U4.C1+
- new net N$22: C4.1, U4.C1-
- new net SCREEN-SDL: U4.SDA
- net 3V3: now also U4.A, U4.RST, U4.VDD
- net GND: now also C5.1, U4.VSS
- net N$3: now also C5.2, U4.VOUT; no longer U$1.A4
- net SCREEN-BLUE: now also U4.K-B; no longer SCREEN.5
- net SCREEN-BLUE-CONTROL: now also SCREEN.5
- net SCREEN-GREEN: now also U4.K-G; no longer SCREEN.7
- net SCREEN-GREEN-CONTROL: now also SCREEN.7
- net SCREEN-RED: now also U4.K-R; no longer SCREEN.9
- net SCREEN-RED-CONTROL: now also SCREEN.9
- net SCREEN-SCL: now also U4.SCL
Other:
- moved on the sheet: R1, R10, R11, R16, R2, R3, R4, R5, R6, R7, R8, R9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

Commit message: Electron Board Changes
Parts:
- removed C4, C5: 1uf, capacitor-wima:C2.5/4
- removed R10, R5, R7: 47k, resistor:R-US_0207/12
- removed R11, R6, R8: 36, resistor:R-US_0207/12
- removed R2, R4, R9: 1k, resistor:R-US_0207/12
- removed SCREEN1: (no value), SparkFun-Connectors:CONN_05X2SHD
- removed T2, T3, T4: 2N2222, transistor:2N2222
- removed U4: NHD‐C0220, GEMS:NHD‐C0220
Connections:
- removed net BLUE-NPN-BASE: R2.2, R5.2, T2.B
- removed net BLUE-NPN-EMITTER: R6.2, T2.E
- removed net GREEN-NPN-BASE: R10.2, R9.2, T4.B
- removed net GREEN-NPN-EMITTER: R11.2, T4.E
- removed net N$21: C4.2, U4.C1+
- removed net N$22: C4.1, U4.C1-
- removed net N$3: C5.2, U4.VOUT
- removed net RED-NPN-BASE: R4.2, R7.2, T3.B
- removed net RED-NPN-EMITTER: R8.2, T3.E
- removed net SCREEN-BLUE: T2.C, U4.K-B
- removed net SCREEN-GREEN: T4.C, U4.K-G
- removed net SCREEN-RED: T3.C, U4.K-R
- removed net SCREEN-SDL: U4.SDA
- net 3V3: no longer U4.A, U4.RST, U4.VDD
- net GND: no longer C5.1, R10.1, R11.1, R5.1, R6.1, R7.1, R8.1, U4.VSS
- net SCREEN-BLUE-CONTROL: no longer R2.1
- net SCREEN-GREEN-CONTROL: no longer R9.1
- net SCREEN-RED-CONTROL: no longer R4.1
- net SCREEN-SCL: no longer U4.SCL
