File: ElectronBoardMKI.brd (EAGLE design)
At the start: 84.2 x 200 mm, 47 parts, among them IC1 7805TV, Q1 BSS170, Q2 BSS170, T2 2N2222, T3 2N2222, T4 2N2222, U1 LM386N

Commit message: Display Board. Attained old board files. Schematic organization.
Parts:
- added C4, C5: 1uf, capacitor-wima:C2.5-4
- added SCREEN1: (no value), SparkFun-Connectors:2X5-SHROUDED
- added U4: NHD‐C0220, GEMS:NHD-C0220
- moved R9 125.2 mm to (66.4, 209.1)
- moved T2 123.0 mm to (69.0, 203.0)
- moved R4 122.9 mm to (11.4, 199.6)
- moved T4 122.1 mm to (60.5, 200.7)
- moved T3 121.2 mm to (52.0, 198.5)
- moved R2 102.9 mm to (62.4, 189.6)
Connections:
- new net N$21: C4.2, U4.7
- new net N$22: C4.1, U4.8
- new net SCREEN-SDL: U4.3
- net 3V3: now also U4.1, U4.5, U4.A
- net GND: now also C5.1, U4.4
- net N$3: now also C5.2, U4.6; no longer U$1.8
- net SCREEN-BLUE: now also U4.BK; no longer SCREEN.5
- net SCREEN-BLUE-CONTROL: now also SCREEN.5
- net SCREEN-GREEN: now also U4.GK; no longer SCREEN.7
- net SCREEN-GREEN-CONTROL: now also SCREEN.7
- net SCREEN-RED: now also U4.RK; no longer SCREEN.9
- net SCREEN-RED-CONTROL: now also SCREEN.9
- net SCREEN-SCL: now also U4.2
Routing:
- net SCREEN-RED: track 28.6 -> 0.00 mm
- net BLUE-NPN-BASE: track 24.8 -> 0.00 mm
- net SCREEN-GREEN: track 17.8 -> 0.00 mm
- net GREEN-NPN-BASE: track 16.3 -> 0.00 mm
- net RED-NPN-BASE: track 15.4 -> 0.64 mm
- net SCREEN-BLUE: track 8.78 -> 0.00 mm
- net BLUE-NPN-EMITTER: track 6.88 -> 0.00 mm
- net GREEN-NPN-EMITTER: track 5.34 -> 0.00 mm
- net SCREEN-BLUE-CONTROL: track 4.34 -> 0.00 mm
- net SCREEN-RED-CONTROL: track 4.34 -> 0.00 mm
- net SCREEN-GREEN-CONTROL: track 4.34 -> 0.00 mm
- net RED-NPN-EMITTER: track 4.07 -> 0.00 mm
- net SCREEN-SCL: track 40.5 -> 41.7 mm
Other:
- board size 84.2 x 200 mm -> 84 x 250 mm

Commit message: Electron Board Changes
Parts:
- removed C4, C5: 1uf, capacitor-wima:C2.5-4
- removed R10, R5, R7: 47k, resistor:0207/12
- removed R11, R6, R8: 36, resistor:0207/12
- removed R2, R4, R9: 1k, resistor:0207/12
- removed SCREEN1: (no value), SparkFun-Connectors:2X5-SHROUDED
- removed T2, T3, T4: 2N2222, transistor:TO18
- removed U4: NHD‐C0220, GEMS:NHD-C0220
- moved C3 36.6 mm to (50.0, 135.3)
- moved R3 36.4 mm to (75.2, 66.4)
- moved R1 35.7 mm to (75.2, 69.8)
- moved SCL___SDA2 34.3 mm to (78.1, 76.2)
- moved SCREEN 29.5 mm to (76.8, 53.0)
- moved R12 28.7 mm to (52.7, 83.8), turned to 270 degrees
- moved C1 23.4 mm to (51.8, 102.6)
- moved IC1 23.4 mm to (62.5, 107.6)
- moved C2 23.2 mm to (77.2, 102.6)
- moved C8 23.2 mm to (75.7, 114.1)
- moved C9 23.2 mm to (74.5, 127.8)
- moved R19 23.2 mm to (82.1, 120.5)
- moved R21 23.2 mm to (54.6, 118.1)
- moved U1 23.2 mm to (65.1, 118.0)
- moved C7 23.2 mm to (64.8, 130.3)
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Connections:
- removed net BLUE-NPN-BASE: R2.2, R5.2, T2.2
- removed net BLUE-NPN-EMITTER: R6.2, T2.1
- removed net GREEN-NPN-BASE: R10.2, R9.2, T4.2
- removed net GREEN-NPN-EMITTER: R11.2, T4.1
- removed net N$21: C4.2, U4.7
- removed net N$22: C4.1, U4.8
- removed net N$3: C5.2, U4.6
- removed net RED-NPN-BASE: R4.2, R7.2, T3.2
- removed net RED-NPN-EMITTER: R8.2, T3.1
- removed net SCREEN-BLUE: T2.3, U4.BK
- removed net SCREEN-GREEN: T4.3, U4.GK
- removed net SCREEN-RED: T3.3, U4.RK
- removed net SCREEN-SDL: U4.3
- net 3V3: no longer U4.1, U4.5, U4.A
- net GND: no longer C5.1, R10.1, R11.1, R5.1, R6.1, R7.1, R8.1, U4.4
- net SCREEN-BLUE-CONTROL: no longer R2.1
- net SCREEN-GREEN-CONTROL: no longer R9.1
- net SCREEN-RED-CONTROL: no longer R4.1
- net SCREEN-SCL: no longer U4.2
Routing:
- net 3V3: track 307.9 -> 233.7 mm
- net SCREEN-BLUE-CONTROL: track 0.00 -> 57.1 mm
- net SCREEN-GREEN-CONTROL: track 0.00 -> 56.9 mm
- net SCREEN-RED-CONTROL: track 0.00 -> 56.9 mm
- net VIN: track 182.7 -> 140.9 mm
- net N$6: track 60.1 -> 32.2 mm
- net SPEAKER-OUTPUT: track 12.9 -> 40.0 mm
- net SCREEN-SCL: track 41.7 -> 59.9 mm
- net SCREEN-SDA: track 42.4 -> 58.4 mm
- net SDA-3V3: track 18.6 -> 24.3 mm
- net SOUND: track 48.3 -> 42.8 mm, vias 1 -> 0
- net SDA-5V: track 34.4 -> 29.3 mm
- net SCL-3V3: track 20.2 -> 17.7 mm
- net SCL-5V: track 31.6 -> 33.8 mm
- net RED-NPN-BASE: track 0.64 -> 0.00 mm
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
Commit message: Final Before Order
Parts:
- added U$3, U$4, U$5, U$6: (no value), holes:4,1
- moved R19 1.27 mm to (80.8, 120.5)
Routing:
- net 3V3: track 233.7 -> 314.0 mm, vias 0 -> 2
- net VIN: track 140.9 -> 197.1 mm, vias 0 -> 1
- net 5V: track 25.2 -> 27.6 mm
- net N$7: track 3.81 -> 2.54 mm
Other:
- board size 84 x 250 mm -> 84 x 200 mm
