File: ArduinoBoardMK1.brd (EAGLE design)
At the start: 95.2 x 82.5 mm, 22 parts, among them K1 AQH2223

Commit message: MKII
Parts:
- R11, R6: value 47k -> 38k
Changed lines of the file:
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@@
 <drawing>
 <settings>
-<setting alwaysvectorfont="yes"/>
+<setting alwaysvectorfont="no"/>
 <setting verticaltext="up"/>
 </settings>
@@
 <attribute name="VALUE" x="2.413" y="48.26" size="0.6096" layer="27" font="vector" ratio="20" rot="R270"/>
 </element>
-<element name="R6" library="resistor" library_urn="urn:adsk.eagle:library:348" package="0207/12" package3d_urn="urn:adsk.eagle:package:25938/1" value="47k" x="37.465" y="44.45" rot="R225">
+<element name="R6" library="resistor" library_urn="urn:adsk.eagle:library:348" package="0207/12" package3d_urn="urn:adsk.eagle:package:25938/1" value="38k" x="37.465" y="44.45" rot="R225">
 <attribute name="NAME" x="40.697890625" y="45.707234375" size="1.27" layer="25" ratio="10" rot="R225"/>
 <attribute name="VALUE" x="38.596509375" y="46.551378125" size="1.27" layer="27" ratio="10" rot="R225"/>
 </element>
-<element name="R11" library="resistor" library_urn="urn:adsk.eagle:library:348" package="0207/12" package3d_urn="urn:adsk.eagle:package:25938/1" value="47k" x="38.1" y="48.895" rot="R45">
+<element name="R11" library="resistor" library_urn="urn:adsk.eagle:library:348" package="0207/12" package3d_urn="urn:adsk.eagle:package:25938/1" value="38k" x="38.1" y="48.895" rot="R45">
 <attribute name="NAME" x="34.86710625" y="47.6377625" size="1.27" layer="25" ratio="10" rot="R45"/>
 <attribute name="VALUE" x="36.9684875" y="46.79361875" size="1.27" layer="27" ratio="10" rot="R45"/>
