File: ElectronBoardMKII.sch (EAGLE design)
At the start: 45 parts, among them IC1 7805TV, K1 AQYAQY27, Q1 BSS170, Q2 BSS170, U1 LM386N

Commit message: More
Parts:
- added C10: 250uF, resistor:CPOL-US085CS-1AR
- added C4: 10uF, resistor:CPOL-US085CS-1AR
- added C5: 1uF, resistor:CPOL-US085CS-1AR
- added C6: 0.05uF, resistor:CPOL-US085CS-1AR
- added IC: LM386M-1, linear:LM386M-1
- added R7: 10K, resistor:R-US_M0805
- added R8, R9: 10K, pot:TRIM_US-3223G
- added SP1: KSS1201, buzzer:KSS1201
Connections:
- new net N$14: C5.+, IC.BYPASS
- new net N$16: C10.+, C6.+, IC.OUT
- new net N$17: C4.-, IC.GAIN@2
- new net N$18: IC.+IN, R8.S
- new net N$19: C6.-, R7.2
- new net N$20: IC.GAIN@1, R9.E
- new net N$21: C4.+, R9.S
- new net VCC: IC.VS
- new net VO: C10.-, SP1.1
- net GND: now also C5.-, IC.-IN, IC.GND, R7.1, R8.A, SP1.2
- net VIN: now also R8.E
Other:
- note added: "Audio signal input from Mic"

Commit message: Electron Side Header Start
Parts:
- added J2, J3, J4, J5, J6: (no value), SparkFun-Connectors:CONN_09LOCK
Connections:
- new net A4: J2.8
- new net A5: J2.7
- new net DAC: J2.6
- new net N$22: J6.1
- new net N$23: J6.2
- new net N$24: J6.3
- new net N$25: J6.4
- new net N$26: J6.5
- new net N$27: J6.6
- new net N$28: J6.7
- new net N$29: J6.8
- new net N$30: J6.9
- new net N$31: U$1.A5
- new net WKP: J2.5
- net COOLING-CURRENT: now also J2.9
- net GND: now also J2.2
- net IN-TEMP: no longer U$1.DAC
- net RX: now also J2.4
- net TX: now also J2.3
- net VIN: now also J2.1
Other:
- moved on the sheet: J1, RX_______TX

Commit message: Progress!
Parts:
- removed C10: 250uF, resistor:CPOL-US085CS-1AR
- removed C5: 1uF, resistor:CPOL-US085CS-1AR
- removed C6: 0.05uF, resistor:CPOL-US085CS-1AR
- removed IC: LM386M-1, linear:LM386M-1
- removed SP1: KSS1201, buzzer:KSS1201
- added J7: (no value), jumper:J2X2MM
- C4: value 10uF -> 1uf; device resistor:CPOL-US085CS-1AR -> resistor:CPOL-USE5-8.5
- J5: device SparkFun-Connectors:CONN_09LOCK -> jumper:J2X2MM
- R2, R4, R5, R6: value 10k -> (none); device resistor:R-US_0207/12 -> adafruit:R-US_0207/10
- R7: value 10K -> (none); device resistor:R-US_M0805 -> adafruit:R-US_0207/10
- R8: value 10K -> 10k; device pot:TRIM_US-3223G -> pot:TRIM_US-CT6
- R9: value 10K -> (none); device pot:TRIM_US-3223G -> resistor:R-US_0207/5V
Connections:
- removed net A5: J2.7
- removed net N$17: C4.-, IC.GAIN@2
- removed net N$18: IC.+IN, R8.S
- removed net N$19: C6.-, R7.2
- removed net N$20: IC.GAIN@1, R9.E
- removed net N$21: C4.+, R9.S
- removed net N$22: J6.1
- removed net N$23: J6.2
- removed net N$24: J6.3
- removed net N$25: J6.4
- removed net N$26: J6.5
- removed net N$27: J6.6
- removed net N$28: J6.7
- removed net N$29: J6.8
- removed net N$30: J6.9
- removed net N$31: U$1.A5
- removed net VCC: IC.VS
- removed net VO: C10.-, SP1.1
- new net A2: J6.1, U$1.A2
- new net D5: J3.7, U$1.D5
- new net D6: J3.6, U$1.D6
- new net D7: J3.5, U$1.D7
- new net LIGHTS: J4.9, K1.A, U$1.C0
- new net RST: J3.2, U$1.!RST
- new net VBAT: J3.3, U$1.VBAT
- net 3V3: now also J3.1, R8.E
- net 5V: now also J5.1
- net A4: now also U$1.A4
- net COOLING-INA: now also J4.1
- net COOLING-INB: now also J3.8
- net COOLING-PWM: now also J3.9
- net DAC: now also J7.3, U$1.DAC
- net GND: now also J3.4; no longer C5.-, IC.-IN, IC.GND, SP1.2
- net IN-TEMP: now also J2.7, U$1.A5
- net KEYPAD-1: now also J6.5
- net KEYPAD-2: now also J6.6
- net KEYPAD-3: now also J6.7
- net KEYPAD-A: now also J6.3
- net KEYPAD-B: now also J6.4
- net KEYPAD-C: now also J6.9
- net KEYPAD-D: now also J6.8
- net N$1: now also C4.+, R9.1; no longer R21.S
- net N$10: now also J5.2
- net N$14: now also C4.-, R21.S; no longer C5.+, IC.BYPASS
- net N$16: now also R8.S, R9.2; no longer C10.+, C6.+, IC.OUT
- net N$8: now also K1.K, R7.2; no longer U$1.D5
- net OUT-TEMP: now also J6.2
- net SCL-3V3: now also J4.2
- net SCREEN-BLUE-CONTROL: now also J4.6
- net SCREEN-GREEN-CONTROL: now also J4.7
- net SCREEN-RED-CONTROL: now also J4.8
- net SCREEN-SCL: now also J4.4
- net SCREEN-SDA: now also J4.5
- net SDA-3V3: now also J4.3
- net SOUND: now also J7.2; no longer U$1.WKP
- net VIN: now also J5.3; no longer R8.E
- net WKP: now also J7.1, U$1.WKP
Other:
- note removed: "Audio signal input from Mic"
- moved on the sheet: C4, R21, R7, R8

Commit message: Buzzer Progress
Parts:
- renumbered R21 to VOLUME, R22 to GAIN, R8 to BIAS, VIN1 to LEDOUT

Commit message: Update
Parts:
- R9: value (none) -> 100k
Changed lines of the file:
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@@
 <part name="SUPPLY5" library="supply1" library_urn="urn:adsk.eagle:library:371" deviceset="GND" device=""/>
 <part name="C4" library="resistor" library_urn="urn:adsk.eagle:library:348" deviceset="CPOL-US" device="E5-8.5" package3d_urn="urn:adsk.eagle:package:25860/1" value="1uf"/>
-<part name="R9" library="resistor" library_urn="urn:adsk.eagle:library:348" deviceset="R-US_" device="0207/5V" package3d_urn="urn:adsk.eagle:package:23502/1"/>
+<part name="R9" library="resistor" library_urn="urn:adsk.eagle:library:348" deviceset="R-US_" device="0207/5V" package3d_urn="urn:adsk.eagle:package:23502/1" value="100k"/>
 <part name="J7" library="jumper" library_urn="urn:adsk.eagle:library:252" deviceset="J2" device="X2MM" package3d_urn="urn:adsk.eagle:package:15506/1"/>
 </parts>
