File: ArduinoBoardMKII.sch (EAGLE design)
At the start: 26 parts

Commit message: Electron Side Header Start
Connections:
- removed net N$12: J3.2, MICRO.A2
- removed net N$2: J4.6, MICRO.5V
- net +5V: now also J4.6, MICRO.5V
- net DOORSWITCH: now also J3.2, MICRO.A2
- net GND: now also GND.1
Changed lines of the file:
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@@
 <part name="J3" library="SparkFun-Connectors" deviceset="CONN_07" device="LOCK"/>
 <part name="J4" library="SparkFun-Connectors" deviceset="CONN_10" device="LOCK"/>
+<part name="GND9" library="supply1" library_urn="urn:adsk.eagle:library:371" deviceset="GND" device=""/>
+<part name="P+6" library="supply1" library_urn="urn:adsk.eagle:library:371" deviceset="+5V" device=""/>
 </parts>
 <sheets>
@@
 <attribute name="NAME" x="-55.88" y="24.892" size="1.778" layer="95" font="vector" rot="R180"/>
 </instance>
+<instance part="GND9" gate="1" x="20.32" y="27.94">
+<attribute name="VALUE" x="17.78" y="25.4" size="1.778" layer="96"/>
+</instance>
+<instance part="P+6" gate="1" x="-88.9" y="35.56" rot="R90">
+<attribute name="VALUE" x="-83.82" y="33.02" size="1.778" layer="96" rot="R180"/>
+</instance>
 </instances>
 <busses>
@@
 <wire x1="58.42" y1="-45.72" x2="66.04" y2="-45.72" width="0.1524" layer="91"/>
 </segment>
+<segment>
+<pinref part="GND" gate="G$1" pin="1"/>
+<wire x1="15.24" y1="30.48" x2="20.32" y2="30.48" width="0.1524" layer="91"/>
+<pinref part="GND9" gate="1" pin="GND"/>
+</segment>
 </net>
 <net name="+12V" class="0">
@@
 <wire x1="40.64" y1="78.74" x2="40.64" y2="83.82" width="0.1524" layer="91"/>
 </segment>
+<segment>
+<pinref part="MICRO" gate="G$1" pin="5V"/>
+<pinref part="J4" gate="J1" pin="6"/>
+<wire x1="-66.04" y1="38.1" x2="-76.2" y2="38.1" width="0.1524" layer="91"/>
+<wire x1="-76.2" y1="38.1" x2="-78.74" y2="35.56" width="0.1524" layer="91"/>
+<wire x1="-93.98" y1="35.56" x2="-86.36" y2="35.56" width="0.1524" layer="91"/>
+<pinref part="P+6" gate="1" pin="+5V"/>
+<wire x1="-86.36" y1="35.56" x2="-78.74" y2="35.56" width="0.1524" layer="91"/>
+<junction x="-86.36" y="35.56"/>
+</segment>
 </net>
 <net name="SCL" class="0">
@@
 <segment>
 <pinref part="MICRO" gate="G$1" pin="VIN"/>
-<label x="-35.56" y="45.72" size="1.778" layer="95"/>
+<label x="-53.34" y="45.72" size="1.778" layer="95"/>
 <wire x1="-93.98" y1="43.18" x2="-86.36" y2="43.18" width="0.1524" layer="91"/>
 <wire x1="-86.36" y1="43.18" x2="-83.82" y2="45.72" width="0.1524" layer="91"/>
@@
 <pinref part="SWITCH" gate="G$1" pin="1"/>
 </segment>
+<segment>
+<pinref part="MICRO" gate="G$1" pin="A2"/>
+<wire x1="-71.12" y1="20.32" x2="-93.98" y2="20.32" width="0.1524" layer="91"/>
+<wire x1="-71.12" y1="20.32" x2="-68.58" y2="17.78" width="0.1524" layer="91"/>
+<pinref part="J3" gate="J1" pin="2"/>
+<wire x1="-68.58" y1="17.78" x2="-66.04" y2="17.78" width="0.1524" layer="91"/>
+<label x="-53.34" y="17.78" size="1.778" layer="95"/>
+</segment>
 </net>
 <net name="POST-OPTO-DIODE" class="0">
@@
 <segment>
 <pinref part="MICRO" gate="G$1" pin="A5"/>
-<label x="-38.1" y="30.48" size="1.778" layer="95"/>
+<label x="-53.34" y="30.48" size="1.778" layer="95"/>
 <pinref part="J4" gate="J1" pin="9"/>
 <wire x1="-66.04" y1="30.48" x2="-68.58" y2="30.48" width="0.1524" layer="91"/>
@@
 <pinref part="MICRO" gate="G$1" pin="A1"/>
 <wire x1="-73.66" y1="17.78" x2="-93.98" y2="17.78" width="0.1524" layer="91"/>
-<label x="-35.56" y="15.24" size="1.778" layer="95"/>
+<label x="-53.34" y="15.24" size="1.778" layer="95"/>
 </segment>
 </net>
@@
 <pinref part="J3" gate="J1" pin="1"/>
 <wire x1="-66.04" y1="20.32" x2="-68.58" y2="22.86" width="0.1524" layer="91"/>
-</segment>
-</net>
-<net name="N$12" class="0">
-<segment>
-<pinref part="MICRO" gate="G$1" pin="A2"/>
-<wire x1="-71.12" y1="20.32" x2="-93.98" y2="20.32" width="0.1524" layer="91"/>
-<wire x1="-71.12" y1="20.32" x2="-68.58" y2="17.78" width="0.1524" layer="91"/>
-<pinref part="J3" gate="J1" pin="2"/>
-<wire x1="-68.58" y1="17.78" x2="-66.04" y2="17.78" width="0.1524" layer="91"/>
 </segment>
 </net>
@@
 </segment>
 </net>
-<net name="N$2" class="0">
-<segment>
-<pinref part="MICRO" gate="G$1" pin="5V"/>
-<pinref part="J4" gate="J1" pin="6"/>
-<wire x1="-66.04" y1="38.1" x2="-76.2" y2="38.1" width="0.1524" layer="91"/>
-<wire x1="-76.2" y1="38.1" x2="-78.74" y2="35.56" width="0.1524" layer="91"/>
-<wire x1="-93.98" y1="35.56" x2="-78.74" y2="35.56" width="0.1524" layer="91"/>
-</segment>
-</net>

Commit message: Progress!
Parts:
- removed R1: 100, resistor:R-US_0207/12
- added LED1: LED-DIP-3, _led-rgb:LED-DIP-3
- added R2, R4: 220, adafruit:R-US_0207/10
- added R5: 100, adafruit:R-US_0207/10
- R3: device resistor:R-US_0207/12 -> adafruit:R-US_0207/10
Connections:
- removed net N$16: J3.6, MICRO.3V
- removed net N$21: J2.2, MICRO.D7
- removed net N$22: J2.3, MICRO.IO8
- new net 3V3: J3.6, MICRO.3V, TEMPERATURE1.3, TEMPERATURE2.3
- new net N$2: LED1.BLUE, R2.2
- new net N$3: LED1.GREEN, R4.2
- new net RGBD-BLUE: J2.3, MICRO.IO8, R2.1
- new net RGBD-GREEN: J2.2, MICRO.D7, R4.1
- net +5V: no longer TEMPERATURE1.3, TEMPERATURE2.3
- net GND: now also LED1.COM-CATHODE, R5.1; no longer R1.1
- net POST-OPTO-DIODE: now also R5.2; no longer R1.2

Commit message: Update
Parts:
- added JP1, JP2: (no value), jumper:JP2E
Connections:
- new net 5V: JP1.1, JP2.1
- new net N$12: JP2.2, R9.2
- new net N$13: JP1.3
- new net N$21: JP2.3
- new net N$4: JP1.2, R10.2
- net +5V: no longer R9.2
- net GND: no longer R10.1
- net MOTOR-IN2: now also R10.1; no longer R10.2
Other:
- moved on the sheet: CPC1718, MOTOR1-1, MOTOR1-2, R10, R5, R7, R8, R9, TLE5205

Commit message: Buzzer Progress
Parts:
- added J5: (no value), SparkFun-Connectors:CONN_02
- added SG1: F/QMB, buzzer:F/QMB
Connections:
- net N$17 renamed BUZZER
- removed net 5V: JP1.1, JP2.1
- removed net N$13: JP1.3
- removed net N$21: JP2.3
- net +5V: now also JP1.1, JP2.1
- net GND: now also JP1.3, JP2.3
Changed lines of the file:
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@@
 <?xml version="1.0" encoding="utf-8"?>
 <!DOCTYPE eagle SYSTEM "eagle.dtd">
-<eagle version="9.1.3">
+<eagle version="9.2.0">
 <drawing>
 <settings>
@@
 <part name="JP1" library="jumper" library_urn="urn:adsk.eagle:library:252" deviceset="JP2E" device="" package3d_urn="urn:adsk.eagle:package:15452/1"/>
 <part name="JP2" library="jumper" library_urn="urn:adsk.eagle:library:252" deviceset="JP2E" device="" package3d_urn="urn:adsk.eagle:package:15452/1"/>
+<part name="GND10" library="supply1" library_urn="urn:adsk.eagle:library:371" deviceset="GND" device=""/>
+<part name="GND15" library="supply1" library_urn="urn:adsk.eagle:library:371" deviceset="GND" device=""/>
+<part name="P+3" library="supply1" library_urn="urn:adsk.eagle:library:371" deviceset="+5V" device=""/>
+<part name="P+5" library="supply1" library_urn="urn:adsk.eagle:library:371" deviceset="+5V" device=""/>
+<part name="SG1" library="buzzer" library_urn="urn:adsk.eagle:library:113" deviceset="F/QMB" device="" package3d_urn="urn:adsk.eagle:package:5270/1"/>
+<part name="J5" library="SparkFun-Connectors" deviceset="CONN_02" device=""/>
 </parts>
 <sheets>
@@
 </instance>
 <instance part="P+4" gate="1" x="5.08" y="-12.7">
-<attribute name="VALUE" x="2.54" y="-5.08" size="1.778" layer="96" rot="R90"/>
+<attribute name="VALUE" x="2.54" y="-17.78" size="1.778" layer="96" rot="R90"/>
 </instance>
 <instance part="MOTOR1" gate="-1" x="20.32" y="-66.04" rot="R180">
@@
 <instance part="J2" gate="J1" x="-160.02" y="15.24" rot="MR180">
 <attribute name="VALUE" x="-165.1" y="25.146" size="1.778" layer="96" font="vector" rot="MR180"/>
-<attribute name="NAME" x="-165.1" y="-0.508" size="1.778" layer="95" font="vector" rot="MR180"/>
+<attribute name="NAME" x="-165.1" y="2.032" size="1.778" layer="95" font="vector" rot="MR180"/>
 </instance>
 <instance part="J3" gate="J1" x="-60.96" y="15.24" rot="R180">
@@
 <attribute name="VALUE" x="-83.82" y="33.02" size="1.778" layer="96" rot="R180"/>
 </instance>
-<instance part="LED1" gate="G$1" x="-129.54" y="-45.72"/>
+<instance part="LED1" gate="G$1" x="-129.54" y="-45.72">
+<attribute name="NAME" x="-137.16" y="-60.198" size="1.778" layer="95"/>
+</instance>
 <instance part="R2" gate="G$1" x="-152.4" y="-40.64">
 <attribute name="NAME" x="-156.21" y="-39.1414" size="1.778" layer="95"/>
@@
 <attribute name="VALUE" x="-34.798" y="-34.29" size="1.778" layer="96" rot="R90"/>
 </instance>
-<instance part="JP1" gate="1" x="-30.48" y="-93.98" rot="MR180"/>
-<instance part="JP2" gate="1" x="-30.48" y="-53.34"/>
+<instance part="JP1" gate="1" x="-30.48" y="-93.98" rot="MR180">
+<attribute name="NAME" x="-34.29" y="-93.98" size="1.778" layer="95" rot="MR270"/>
+<attribute name="VALUE" x="-24.765" y="-93.98" size="1.778" layer="96" rot="MR270"/>
+</instance>
+<instance part="JP2" gate="1" x="-30.48" y="-53.34">
+<attribute name="NAME" x="-34.29" y="-53.34" size="1.778" layer="95" rot="R90"/>
+<attribute name="VALUE" x="-24.765" y="-53.34" size="1.778" layer="96" rot="R90"/>
+</instance>
+<instance part="GND10" gate="1" x="-25.4" y="-93.98">
+<attribute name="VALUE" x="-27.94" y="-96.52" size="1.778" layer="96"/>
+</instance>
+<instance part="GND15" gate="1" x="-25.4" y="-60.96">
+<attribute name="VALUE" x="-27.94" y="-63.5" size="1.778" layer="96"/>
+</instance>
+<instance part="P+3" gate="1" x="-40.64" y="-58.42" rot="R90">
+<attribute name="VALUE" x="-35.56" y="-60.96" size="1.778" layer="96" rot="R180"/>
+</instance>
+<instance part="P+5" gate="1" x="-40.64" y="-91.44" rot="R90">
+<attribute name="VALUE" x="-35.56" y="-93.98" size="1.778" layer="96" rot="R180"/>
+</instance>
+<instance part="SG1" gate="G$1" x="-121.92" y="-10.16">
+<attribute name="NAME" x="-124.46" y="-3.81" size="1.778" layer="95"/>
+<attribute name="VALUE" x="-115.57" y="-10.16" size="1.778" layer="96"/>
+</instance>
+<instance part="J5" gate="G$1" x="-182.88" y="-12.7">
+<attribute name="VALUE" x="-185.42" y="-17.526" size="1.778" layer="96" font="vector"/>
+<attribute name="NAME" x="-185.42" y="-7.112" size="1.778" layer="95" font="vector"/>
+</instance>
 </instances>
 <busses>
@@
 <pinref part="GND11" gate="1" pin="GND"/>
 </segment>
+<segment>
+<pinref part="JP1" gate="1" pin="3"/>
+<wire x1="-27.94" y1="-91.44" x2="-25.4" y2="-91.44" width="0.1524" layer="91"/>
+<pinref part="GND10" gate="1" pin="GND"/>
+</segment>
+<segment>
+<pinref part="JP2" gate="1" pin="3"/>
+<wire x1="-27.94" y1="-55.88" x2="-27.94" y2="-58.42" width="0.1524" layer="91"/>
+<wire x1="-27.94" y1="-58.42" x2="-25.4" y2="-58.42" width="0.1524" layer="91"/>
+<pinref part="GND15" gate="1" pin="GND"/>
+</segment>
 </net>
 <net name="+12V" class="0">
@@
 <junction x="-86.36" y="35.56"/>
 </segment>
+<segment>
+<pinref part="JP2" gate="1" pin="1"/>
+<wire x1="-33.02" y1="-55.88" x2="-33.02" y2="-58.42" width="0.1524" layer="91"/>
+<wire x1="-33.02" y1="-58.42" x2="-38.1" y2="-58.42" width="0.1524" layer="91"/>
+<pinref part="P+3" gate="1" pin="+5V"/>
+</segment>
+<segment>
+<pinref part="JP1" gate="1" pin="1"/>
+<wire x1="-33.02" y1="-91.44" x2="-38.1" y2="-91.44" width="0.1524" layer="91"/>
+<pinref part="P+5" gate="1" pin="+5V"/>
+</segment>
 </net>
 <net name="SCL" class="0">
@@
 </segment>
 </net>
-<net name="N$17" class="0">
+<net name="BUZZER" class="0">
 <segment>
 <pinref part="J3" gate="J1" pin="7"/>
@@
 <pinref part="MICRO" gate="G$1" pin="IO13*"/>
 <wire x1="-83.82" y1="7.62" x2="-93.98" y2="7.62" width="0.1524" layer="91"/>
+<label x="-55.88" y="5.08" size="1.27" layer="95" xref="yes"/>
 </segment>
 </net>
@@
 </segment>
 </net>
-<net name="N$13" class="0">
-<segment>
-<pinref part="JP1" gate="1" pin="3"/>
-<wire x1="-27.94" y1="-91.44" x2="-25.4" y2="-91.44" width="0.1524" layer="91"/>
-<label x="-25.4" y="-91.44" size="1.778" layer="95" xref="yes"/>
-</segment>
-</net>
-<net name="N$21" class="0">
-<segment>
-<pinref part="JP2" gate="1" pin="3"/>
-<wire x1="-27.94" y1="-55.88" x2="-27.94" y2="-58.42" width="0.1524" layer="91"/>
-<wire x1="-27.94" y1="-58.42" x2="-25.4" y2="-58.42" width="0.1524" layer="91"/>
-<label x="-25.4" y="-48.26" size="1.778" layer="95" xref="yes"/>
-</segment>
-</net>
-<net name="5V" class="0">
-<segment>
-<pinref part="JP2" gate="1" pin="1"/>
-<wire x1="-33.02" y1="-55.88" x2="-33.02" y2="-58.42" width="0.1524" layer="91"/>
-<wire x1="-33.02" y1="-58.42" x2="-38.1" y2="-58.42" width="0.1524" layer="91"/>
-<label x="-38.1" y="-58.42" size="1.778" layer="95" rot="R180" xref="yes"/>
-</segment>
-<segment>
-<pinref part="JP1" gate="1" pin="1"/>
-<wire x1="-33.02" y1="-91.44" x2="-38.1" y2="-91.44" width="0.1524" layer="91"/>
-<label x="-38.1" y="-91.44" size="1.778" layer="95" rot="R180" xref="yes"/>
-</segment>
-</net>

Commit message: Update
Parts:
- added R1: 1k, rcl:R-US_0207/7
- added T1: 2N2222, transistor:2N2222
- R11, R6: value 38k -> 47k
- R5: value 100 -> 330
Connections:
- new net N$13: SG1.+, T1.C
- new net N$17: R1.2, T1.B
- net +5V: now also SG1.-
- net BUZZER: now also R1.1
- net GND: now also T1.E
Other:
- moved on the sheet: SG1
Changed lines of the file:
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@@
 <part name="TEMPERATURE2" library="SparkFun-Connectors" library_urn="urn:adsk.eagle:library:513" deviceset="CONN_03" device="LONGPADS" package3d_urn="urn:adsk.eagle:package:38068/1"/>
 <part name="GND12" library="supply1" library_urn="urn:adsk.eagle:library:371" deviceset="GND" device=""/>
-<part name="R6" library="resistor" library_urn="urn:adsk.eagle:library:348" deviceset="R-US_" device="0207/12" package3d_urn="urn:adsk.eagle:package:25938/1" value="38k"/>
-<part name="R11" library="resistor" library_urn="urn:adsk.eagle:library:348" deviceset="R-US_" device="0207/12" package3d_urn="urn:adsk.eagle:package:25938/1" value="38k"/>
+<part name="R6" library="resistor" library_urn="urn:adsk.eagle:library:348" deviceset="R-US_" device="0207/12" package3d_urn="urn:adsk.eagle:package:25938/1" value="47k"/>
+<part name="R11" library="resistor" library_urn="urn:adsk.eagle:library:348" deviceset="R-US_" device="0207/12" package3d_urn="urn:adsk.eagle:package:25938/1" value="47k"/>
 <part name="GND13" library="supply1" library_urn="urn:adsk.eagle:library:371" deviceset="GND" device=""/>
 <part name="GND14" library="supply1" library_urn="urn:adsk.eagle:library:371" deviceset="GND" device=""/>
@@
 <part name="R4" library="adafruit" deviceset="R-US_" device="0207/10" value="220"/>
 <part name="GND11" library="supply1" library_urn="urn:adsk.eagle:library:371" deviceset="GND" device=""/>
-<part name="R5" library="adafruit" deviceset="R-US_" device="0207/10" value="100"/>
+<part name="R5" library="adafruit" deviceset="R-US_" device="0207/10" value="330"/>
 <part name="JP1" library="jumper" library_urn="urn:adsk.eagle:library:252" deviceset="JP2E" device="" package3d_urn="urn:adsk.eagle:package:15452/1"/>
 <part name="JP2" library="jumper" library_urn="urn:adsk.eagle:library:252" deviceset="JP2E" device="" package3d_urn="urn:adsk.eagle:package:15452/1"/>
@@
 <part name="SG1" library="buzzer" library_urn="urn:adsk.eagle:library:113" deviceset="F/QMB" device="" package3d_urn="urn:adsk.eagle:package:5270/1"/>
 <part name="J5" library="SparkFun-Connectors" deviceset="CONN_02" device=""/>
+<part name="T1" library="transistor" library_urn="urn:adsk.eagle:library:402" deviceset="2N2222" device="" package3d_urn="urn:adsk.eagle:package:29892/2"/>
+<part name="R1" library="rcl" library_urn="urn:adsk.eagle:library:334" deviceset="R-US_" device="0207/7" package3d_urn="urn:adsk.eagle:package:23493/1" value="1k"/>
+<part name="GND16" library="supply1" library_urn="urn:adsk.eagle:library:371" deviceset="GND" device=""/>
+<part name="P+7" library="supply1" library_urn="urn:adsk.eagle:library:371" deviceset="+5V" device=""/>
 </parts>
 <sheets>
@@
 <attribute name="VALUE" x="-35.56" y="-93.98" size="1.778" layer="96" rot="R180"/>
 </instance>
-<instance part="SG1" gate="G$1" x="-121.92" y="-10.16">
-<attribute name="NAME" x="-124.46" y="-3.81" size="1.778" layer="95"/>
-<attribute name="VALUE" x="-115.57" y="-10.16" size="1.778" layer="96"/>
+<instance part="SG1" gate="G$1" x="-88.9" y="-12.7" rot="R90">
+<attribute name="NAME" x="-95.25" y="-15.24" size="1.778" layer="95" rot="R90"/>
+<attribute name="VALUE" x="-88.9" y="-6.35" size="1.778" layer="96" rot="R90"/>
 </instance>
 <instance part="J5" gate="G$1" x="-182.88" y="-12.7">
 <attribute name="VALUE" x="-185.42" y="-17.526" size="1.778" layer="96" font="vector"/>
 <attribute name="NAME" x="-185.42" y="-7.112" size="1.778" layer="95" font="vector"/>
+</instance>
+<instance part="T1" gate="G$1" x="-88.9" y="-25.4">
+<attribute name="NAME" x="-99.06" y="-17.78" size="1.778" layer="95"/>
+<attribute name="VALUE" x="-99.06" y="-20.32" size="1.778" layer="96"/>
+</instance>
+<instance part="R1" gate="G$1" x="-99.06" y="-25.4">
+<attribute name="NAME" x="-102.87" y="-23.9014" size="1.778" layer="95"/>
+<attribute name="VALUE" x="-102.87" y="-28.702" size="1.778" layer="96"/>
+</instance>
+<instance part="GND16" gate="1" x="-86.36" y="-38.1">
+<attribute name="VALUE" x="-88.9" y="-40.64" size="1.778" layer="96"/>
+</instance>
+<instance part="P+7" gate="1" x="-86.36" y="-2.54">
+<attribute name="VALUE" x="-86.36" y="-2.54" size="1.778" layer="96"/>
 </instance>
 </instances>
@@
 <pinref part="GND15" gate="1" pin="GND"/>
 </segment>
+<segment>
+<pinref part="T1" gate="G$1" pin="E"/>
+<wire x1="-86.36" y1="-30.48" x2="-86.36" y2="-35.56" width="0.1524" layer="91"/>
+<pinref part="GND16" gate="1" pin="GND"/>
+</segment>
 </net>
 <net name="+12V" class="0">
@@
 <wire x1="-86.36" y1="35.56" x2="-78.74" y2="35.56" width="0.1524" layer="91"/>
 <junction x="-86.36" y="35.56"/>
+<wire x1="-93.98" y1="35.56" x2="-86.36" y2="35.56" width="0.1524" layer="91"/>
 </segment>
 <segment>
@@
 <wire x1="-33.02" y1="-91.44" x2="-38.1" y2="-91.44" width="0.1524" layer="91"/>
 <pinref part="P+5" gate="1" pin="+5V"/>
+</segment>
+<segment>
+<pinref part="SG1" gate="G$1" pin="-"/>
+<wire x1="-86.36" y1="-7.62" x2="-86.36" y2="-5.08" width="0.1524" layer="91"/>
+<pinref part="P+7" gate="1" pin="+5V"/>
 </segment>
 </net>
@@
 <net name="BUZZER" class="0">
 <segment>
-<pinref part="J3" gate="J1" pin="7"/>
-<wire x1="-66.04" y1="5.08" x2="-81.28" y2="5.08" width="0.1524" layer="91"/>
 <wire x1="-81.28" y1="5.08" x2="-83.82" y2="7.62" width="0.1524" layer="91"/>
 <pinref part="MICRO" gate="G$1" pin="IO13*"/>
 <wire x1="-83.82" y1="7.62" x2="-93.98" y2="7.62" width="0.1524" layer="91"/>
+<pinref part="J3" gate="J1" pin="7"/>
+<wire x1="-81.28" y1="5.08" x2="-66.04" y2="5.08" width="0.1524" layer="91"/>
 <label x="-55.88" y="5.08" size="1.27" layer="95" xref="yes"/>
+</segment>
+<segment>
+<pinref part="R1" gate="G$1" pin="1"/>
+<wire x1="-104.14" y1="-25.4" x2="-109.22" y2="-25.4" width="0.1524" layer="91"/>
+<label x="-109.22" y="-25.4" size="1.27" layer="95" rot="R180" xref="yes"/>
 </segment>
 </net>
@@
 <wire x1="-30.48" y1="-55.88" x2="-30.48" y2="-58.42" width="0.1524" layer="91"/>
 <pinref part="JP2" gate="1" pin="2"/>
+</segment>
+</net>
+<net name="N$13" class="0">
+<segment>
+<pinref part="T1" gate="G$1" pin="C"/>
+<pinref part="SG1" gate="G$1" pin="+"/>
+<wire x1="-86.36" y1="-20.32" x2="-86.36" y2="-15.24" width="0.1524" layer="91"/>
+</segment>
+</net>
+<net name="N$17" class="0">
+<segment>
+<pinref part="R1" gate="G$1" pin="2"/>
+<pinref part="T1" gate="G$1" pin="B"/>
+<wire x1="-93.98" y1="-25.4" x2="-91.44" y2="-25.4" width="0.1524" layer="91"/>
 </segment>
 </net>
@@
 packages will not be understood (or retained) with this version.
 </note>
+<note version="8.4" severity="warning">
+Since Version 8.4, EAGLE supports properties for SPICE simulation.
+Probes in schematics and SPICE mapping objects found in parts and library devices
+will not be understood with this version. Update EAGLE to the latest version
+for full support of SPICE simulation.
+</note>
 </compatibility>

Commit message: Updated Arduino wih correct grounding and board size.
Parts:
- removed J5: (no value), SparkFun-Connectors:CONN_02
- added J6: (no value), SparkFun-Connectors:CONN_021X02_NO_SILK
- R1: value 1k -> 220; device rcl:R-US_0207/7 -> adafruit:R-US_0207/10
- R10: value 47k -> 1k; device resistor:R-US_0207/12 -> rcl:R-US_0207/7
- R11: value 47k -> 4.7k; device resistor:R-US_0207/12 -> adafruit:R-US_0207/10
- R3: value 4.7k -> 330
- R4: value 220 -> 47k; device adafruit:R-US_0207/10 -> resistor:R-US_0207/10
- R5: value 330 -> 47k; device adafruit:R-US_0207/10 -> resistor:R-US_0207/10
Connections:
- removed net N$1: J4.4, MICRO.GND1
- removed net N$5: J1.6, MICRO.GND
- net +5V: now also J6.2
- net BUZZER: now also R10.1; no longer R1.1
- net DOORSWITCH: now also R11.1; no longer R3.1
- net GND: now also J1.6, J4.4, MICRO.GND, MICRO.GND1, R3.1, R4.2; no longer R3.2, R6.1
- net IN1: now also R8.2; no longer R7.2
- net IN2: now also R7.2; no longer R8.2
- net MOTOR-IN1: now also R8.1; no longer R7.1
- net MOTOR-IN2: now also R6.1, R7.1; no longer R10.1, R8.1
- net N$13: now also J6.1
- net N$17: now also R10.2; no longer R1.2
- net N$3: now also R1.2; no longer R4.2
- net N$4: now also R6.2; no longer R10.2
- net PELTIER-INA: now also R4.1; no longer R11.1
- net PELTIER-INB: now also R5.2; no longer R6.2
- net POST-OPTO-DIODE: now also R3.2; no longer R5.2
- net RGBD-GREEN: now also R1.1; no longer R4.1
Other:
- moved on the sheet: R1, R10, R11, R3, R4, R5, R6, R7, R8
