File: ElectronBoardMKII.brd (EAGLE design)
At the start: 84 x 200 mm, 63 parts, among them IC1 7805TV, K1 AQYAQY27, Q1 BSS170, Q2 BSS170, U1 LM386N

Commit message: Progress!
Parts:
- removed C10: 250uF, resistor:085CS_1AR
- removed C5: 1uF, resistor:085CS_1AR
- removed C6: 0.05uF, resistor:085CS_1AR
- removed IC: LM386M-1, linear:SO08
- removed SP1: KSS1201, buzzer:KSS1201
- added J7: (no value), jumper:04C
- C4: value 10uF -> 1uf; device resistor:085CS_1AR -> resistor:E5-8,5
- J5: device SparkFun-Connectors:1X09_LOCK -> jumper:04C
- R2, R4, R5, R6: value 10k -> (none); device resistor:0207/12 -> adafruit:0207/10
- R7: value 10K -> (none); device resistor:M0805 -> adafruit:0207/10
- R8: value 10K -> 10k; device pot:3223G -> pot:CT6
- R9: value 10K -> (none); device pot:3223G -> resistor:0207/5V
- moved J3 238.6 mm to (37.1, 124.5), turned to 270 degrees
- moved J5 230.3 mm to (64.5, 98.4), turned to 180 degrees
- moved J2 229.2 mm to (11.4, 124.5), turned to 270 degrees
- moved J6 221.7 mm to (11.4, 101.6), turned to 270 degrees
- moved J4 220.3 mm to (37.1, 101.6), turned to 270 degrees
- moved R8 202.3 mm to (47.3, 130.2), turned to 90 degrees
- moved R9 194.1 mm to (55.9, 121.0), turned to 180 degrees
- moved C4 180.9 mm to (65.4, 118.4), flipped to the bottom, turned to 270 degrees
- moved R7 125.1 mm to (48.3, 53.3), turned to 270 degrees
- moved R15 9.84 mm to (74.0, 90.2)
- moved R19 8.94 mm to (81.8, 129.4)
- moved VIN1 8.91 mm to (76.2, 35.6)
- moved U1 8.89 mm to (74.0, 118.0)
- moved C3 7.68 mm to (57.6, 136.2)
- moved R16 6.75 mm to (36.2, 71.1)
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Connections:
- removed net A5: J2.7
- removed net N$17: C4.-, IC.8
- removed net N$18: IC.3, R8.2
- removed net N$19: C6.-, R7.2
- removed net N$20: IC.1, R9.3
- removed net N$21: C4.+, R9.2
- removed net N$22: J6.1
- removed net N$23: J6.2
- removed net N$24: J6.3
- removed net N$25: J6.4
- removed net N$26: J6.5
- removed net N$27: J6.6
- removed net N$28: J6.7
- removed net N$29: J6.8
- removed net N$30: J6.9
- removed net N$31: U$1.7
- removed net VCC: IC.6
- removed net VO: C10.-, SP1.+
- new net A2: J6.1, U$1.10
- new net D5: J3.7, U$1.30
- new net D6: J3.6, U$1.31
- new net D7: J3.5, U$1.32
- new net LIGHTS: J4.9, K1.1, U$1.19
- new net RST: J3.2, U$1.35
- net 3V3: now also J3.1, R8.E
- net 5V: now also J5.1
- net A4: now also U$1.8
- net COOLING-INA: now also J4.1
- net COOLING-INB: now also J3.8
- net COOLING-PWM: now also J3.9
- net DAC: now also J7.3, U$1.6
- net GND: now also J3.4, R8.A; no longer C5.-, IC.2, IC.4, R8.1, SP1.-
- net IN-TEMP: now also J2.7, U$1.7
- net KEYPAD-1: now also J6.5
- net KEYPAD-2: now also J6.6
- net KEYPAD-3: now also J6.7
- net KEYPAD-A: now also J6.3
- net KEYPAD-B: now also J6.4
- net KEYPAD-C: now also J6.9
- net KEYPAD-D: now also J6.8
- net N$1: now also C4.+, R9.1; no longer R21.S
- net N$10: now also J5.2
- net N$14: now also C4.-, R21.S; no longer C5.+, IC.7
- net N$16: now also R8.S, R9.2; no longer C10.+, C6.+, IC.5
- net N$8: now also K1.2, R7.2; no longer U$1.30
- net OUT-TEMP: now also J6.2
- net SCL-3V3: now also J4.2
- net SCREEN-BLUE-CONTROL: now also J4.6
- net SCREEN-GREEN-CONTROL: now also J4.7
- net SCREEN-RED-CONTROL: now also J4.8
- net SCREEN-SCL: now also J4.4
- net SCREEN-SDA: now also J4.5
- net SDA-3V3: now also J4.3
- net SOUND: now also J7.2; no longer U$1.5
- net VBAT: now also J3.3
- net VIN: now also J5.3; no longer R8.3
- net WKP: now also J7.1, U$1.5
Routing:
- net N$11: track 0.00 -> 43.1 mm
- net DAC: track 0.00 -> 36.4 mm
- net LIGHTS: track 0.00 -> 36.4 mm
- net N$10: track 0.00 -> 35.8 mm
- net WKP: track 0.00 -> 29.7 mm
- net COOLING-OUTA: track 28.8 -> 54.0 mm
- net VIN: track 197.1 -> 220.3 mm
- net 3V3: track 315.2 -> 337.7 mm, vias 2 -> 0
- net COOLING-OUTB: track 34.4 -> 45.9 mm
- net +12V: track 15.0 -> 26.5 mm
- net SOUND: track 42.8 -> 31.5 mm
- net N$16: track 0.00 -> 10.7 mm
- net N$8: track 0.00 -> 9.88 mm
- net IN-TEMP: track 0.00 -> 9.78 mm
- net SCL-3V3: track 17.7 -> 27.2 mm
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
Commit message: Update
Parts:
- moved R1 0.32 mm to (75.2, 70.2)
- moved R3 0.32 mm to (75.2, 66.0)
Changed lines of the file:
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@@
 <attribute name="VALUE" x="3.1115" y="93.218" size="0.6096" layer="27" font="vector" ratio="20" rot="R270"/>
 </element>
-<element name="R1" library="resistor" library_urn="urn:adsk.eagle:library:348" package="0207/12" package3d_urn="urn:adsk.eagle:package:23489/1" value="4.7k" x="75.2475" y="69.85">
-<attribute name="NAME" x="72.0725" y="71.247" size="1.27" layer="25" ratio="10"/>
-<attribute name="VALUE" x="72.9615" y="69.1642" size="1.27" layer="27" ratio="10"/>
-</element>
-<element name="R3" library="resistor" library_urn="urn:adsk.eagle:library:348" package="0207/12" package3d_urn="urn:adsk.eagle:package:23489/1" value="4.7k" x="75.2475" y="66.3575">
-<attribute name="NAME" x="72.0725" y="67.7545" size="1.27" layer="25" ratio="10"/>
-<attribute name="VALUE" x="72.9615" y="65.6717" size="1.27" layer="27" ratio="10"/>
+<element name="R1" library="resistor" library_urn="urn:adsk.eagle:library:348" package="0207/12" package3d_urn="urn:adsk.eagle:package:23489/1" value="4.7k" x="75.2475" y="70.1675">
+<attribute name="NAME" x="72.0725" y="71.5645" size="1.27" layer="25" ratio="10"/>
+<attribute name="VALUE" x="72.9615" y="69.4817" size="1.27" layer="27" ratio="10"/>
+</element>
+<element name="R3" library="resistor" library_urn="urn:adsk.eagle:library:348" package="0207/12" package3d_urn="urn:adsk.eagle:package:23489/1" value="4.7k" x="75.2475" y="66.04">
+<attribute name="NAME" x="72.0725" y="67.437" size="1.27" layer="25" ratio="10"/>
+<attribute name="VALUE" x="72.9615" y="65.3542" size="1.27" layer="27" ratio="10"/>
 </element>
 <element name="R16" library="resistor" library_urn="urn:adsk.eagle:library:348" package="0207/12" package3d_urn="urn:adsk.eagle:package:23489/1" value="47k" x="36.195" y="71.12" rot="R90">
@@
 <contactref element="SCREEN" pad="2"/>
 <contactref element="R3" pad="1"/>
-<wire x1="68.8975" y1="66.3575" x2="69.85" y2="66.3575" width="0.635" layer="16"/>
-<wire x1="69.85" y1="66.3575" x2="78.105" y2="58.1025" width="0.635" layer="16"/>
+<wire x1="68.8975" y1="66.04" x2="70.1675" y2="66.04" width="0.635" layer="16"/>
+<wire x1="70.1675" y1="66.04" x2="78.105" y2="58.1025" width="0.635" layer="16"/>
 <wire x1="39.37" y1="91.44" x2="47.3075" y2="83.5025" width="0.635" layer="1"/>
 <wire x1="47.3075" y1="83.5025" x2="47.3075" y2="73.9775" width="0.635" layer="1"/>
-<wire x1="47.3075" y1="73.9775" x2="54.9275" y2="66.3575" width="0.635" layer="1"/>
-<wire x1="54.9275" y1="66.3575" x2="68.8975" y2="66.3575" width="0.635" layer="1"/>
+<wire x1="47.3075" y1="73.9775" x2="55.245" y2="66.04" width="0.635" layer="1"/>
+<wire x1="55.245" y1="66.04" x2="68.8975" y2="66.04" width="0.635" layer="1"/>
 <contactref element="J4" pad="5"/>
 <wire x1="37.2745" y1="91.44" x2="39.37" y2="91.44" width="0.635" layer="1"/>
@@
 <contactref element="SCREEN" pad="1"/>
 <contactref element="R1" pad="1"/>
-<wire x1="75.565" y1="58.1025" x2="75.565" y2="63.1825" width="0.635" layer="1"/>
-<wire x1="75.565" y1="63.1825" x2="68.8975" y2="69.85" width="0.635" layer="1"/>
-<wire x1="68.8975" y1="69.85" x2="53.975" y2="69.85" width="0.635" layer="1"/>
+<wire x1="75.565" y1="58.1025" x2="75.565" y2="63.5" width="0.635" layer="1"/>
+<wire x1="75.565" y1="63.5" x2="68.8975" y2="70.1675" width="0.635" layer="1"/>
+<wire x1="68.8975" y1="70.1675" x2="53.6575" y2="70.1675" width="0.635" layer="1"/>
 <wire x1="39.37" y1="93.98" x2="48.9331" y2="84.4169" width="0.635" layer="1"/>
-<wire x1="53.975" y1="69.85" x2="48.9331" y2="74.8919" width="0.635" layer="1"/>
+<wire x1="53.6575" y1="70.1675" x2="48.9331" y2="74.8919" width="0.635" layer="1"/>
 <wire x1="48.9331" y1="74.8919" x2="48.9331" y2="84.4169" width="0.635" layer="1"/>
 <contactref element="J4" pad="4"/>
@@
 <wire x1="78.105" y1="53.0225" x2="79.6925" y2="53.0225" width="1.27" layer="1"/>
 <wire x1="79.6925" y1="53.0225" x2="81.5975" y2="54.9275" width="1.27" layer="1"/>
-<wire x1="81.5975" y1="54.9275" x2="81.5975" y2="66.3575" width="1.27" layer="1"/>
-<wire x1="81.5975" y1="66.3575" x2="81.5975" y2="69.85" width="1.27" layer="1"/>
+<wire x1="81.5975" y1="54.9275" x2="81.5975" y2="66.04" width="1.27" layer="1"/>
+<wire x1="81.5975" y1="66.04" x2="81.5975" y2="70.1675" width="1.27" layer="1"/>
 <wire x1="52.705" y1="77.47" x2="54.9275" y2="77.47" width="1.27" layer="1"/>
 <wire x1="54.9275" y1="77.47" x2="57.785" y2="80.3275" width="1.27" layer="1"/>
 <wire x1="57.785" y1="80.3275" x2="57.785" y2="81.915" width="1.27" layer="1"/>
 <wire x1="57.785" y1="80.3275" x2="65.7225" y2="72.39" width="1.27" layer="1"/>
-<wire x1="65.7225" y1="72.39" x2="79.0575" y2="72.39" width="1.27" layer="1"/>
-<wire x1="79.0575" y1="72.39" x2="81.5975" y2="69.85" width="1.27" layer="1"/>
+<wire x1="65.7225" y1="72.39" x2="79.375" y2="72.39" width="1.27" layer="1"/>
+<wire x1="79.375" y1="72.39" x2="81.5975" y2="70.1675" width="1.27" layer="1"/>
 <wire x1="81.5975" y1="46.99" x2="81.5975" y2="51.1175" width="1.27" layer="1"/>
 <wire x1="81.5975" y1="51.1175" x2="79.6925" y2="53.0225" width="1.27" layer="1"/>

Commit message: Buzzer Progress
Parts:
- removed R8: 10k, pot:CT6
- added BIAS: 10k, pot:CT6
- moved C9 2.13 mm to (75.1, 131.6)
- flipped C4 to the top
- renumbered R21 to VOLUME, R22 to GAIN, VIN1 to LEDOUT
Connections:
- net 3V3: now also BIAS.E; no longer R8.E
- net GND: now also BIAS.A; no longer R8.A
- net N$16: now also BIAS.S; no longer R8.S
Routing:
- net 3V3: track 337.9 -> 333.0 mm
- net N$2: track 11.0 -> 12.7 mm
- net N$16: track 10.7 -> 11.4 mm
- net N$1: vias 0 -> 1
Other:
- board text added: "+ -"

Commit message: Update
Parts:
- R9: value (none) -> 100k
Changed lines of the file:
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@@
 <drawing>
 <settings>
-<setting alwaysvectorfont="yes"/>
+<setting alwaysvectorfont="no"/>
 <setting verticaltext="up"/>
 </settings>
@@
 <attribute name="VALUE" x="62.3824" y="120.9421" size="1.27" layer="27" ratio="10" rot="R270"/>
 </element>
-<element name="R9" library="resistor" library_urn="urn:adsk.eagle:library:348" package="0207/5V" package3d_urn="urn:adsk.eagle:package:23502/1" value="" x="55.88" y="120.9675" rot="R180">
+<element name="R9" library="resistor" library_urn="urn:adsk.eagle:library:348" package="0207/5V" package3d_urn="urn:adsk.eagle:package:23502/1" value="100k" x="55.88" y="120.9675" rot="R180">
 <attribute name="NAME" x="57.023" y="120.0785" size="1.27" layer="25" ratio="10" rot="R180"/>
 <attribute name="VALUE" x="57.023" y="123.1265" size="1.27" layer="27" ratio="10" rot="R180"/>
