File: NHD/DisplayBoardMk1.sch (EAGLE design)
At the start: 24 parts

Commit message: Display Board. Attained old board files. Schematic organization.
Parts:
- removed 12V, MOTOR1, PELTIER1, VIN: SMKDSP_1,5/2, con-phoenix-smkdsp:SMKDSP_1,5/2
- removed D2: 1N4004, diode:1N4004
- removed MICRO: ARDUINO_MICROFOOTPRINT, arduino-micro:ARDUINO_MICROFOOTPRINT
- removed PC817: PC817, optocoupler:PC817
- removed R1: 220, resistor:R-US_0207/12
- removed R3: 4.7k, resistor:R-US_0207/12
- removed RELAY: G5LE, relay:G5LE
- removed SDA__SCL1, SDA__SCL2, SWITCH: (no value), SparkFun-Connectors:CONN_02PTH3
- removed TEMPERATURE1, TEMPERATURE2: (no value), SparkFun-Connectors:CONN_03LONGPADS
- removed TLE5205: TLE5205-2, infineon:TLE5205-2
- removed VNH5019: VNH5019VNH5019BOARD, GEMS:VNH5019VNH5019BOARD
- added C4, C5: 0.1uf, capacitor-wima:C2.5/4
- added R4: 1k, resistor:R-US_0207/12
- added R5: 47k, resistor:R-US_0207/12
- added SCREEN: (no value), SparkFun-Connectors:CONN_05X2SHD
- added T2, T3, T4: 2N2222, transistor:2N2222
- added U4: NHD‐C0220, GEMS:NHD‐C0220
- R11, R6: value 47k -> 36
- R2: value 220 -> 1k
- R7: value 1k -> 47k
- R8: value 1k -> 36
- R9: value 47k -> 1k
Connections:
- removed net +12V: 12V-1.KL, R2.2, RELAY2.S, VNH5019.VIN1, VNH5019.VIN2
- removed net +5V: MICRO.5V, R9.2, SWITCH.2, TEMPERATURE1.3, TEMPERATURE2.3, VNH5019.VDD
- removed net DOORSWITCH: MICRO.A2, R3.1, SWITCH.1
- removed net FLYBACK-DIODE+: D2.C, R2.1, RELAY1.1
- removed net IN1: R7.2, TLE5205.IN1
- removed net IN2: R8.2, TLE5205.IN2
- removed net MOTOR-ENABLE: MICRO.IO9*, PC817.A
- removed net MOTOR-ERRORFLAG: MICRO.IO12*, TLE5205.EF
- removed net MOTOR-IN1: MICRO.IO10*, R7.1, R9.1
- removed net MOTOR-IN2: MICRO.IO11*, R10.2, R8.1
- removed net MOTOR-OUT1: MOTOR1-1.KL, TLE5205.OUT1
- removed net MOTOR-OUT2: MOTOR1-2.KL, TLE5205.OUT2
- removed net PELTIER-CURRENT: MICRO.A0, VNH5019.CS
- removed net PELTIER-INA: MICRO.D6*, R11.1, VNH5019.INA
- removed net PELTIER-INB: MICRO.D4*, R6.2, VNH5019.INB
- removed net PELTIER-OUTA: PELTIER1-2.KL, VNH5019.OUTA1, VNH5019.OUTA2
- removed net PELTIER-OUTB: PELTIER1-1.KL, VNH5019.OUTB1, VNH5019.OUTB2
- removed net PELTIER-PWM: MICRO.D5*, VNH5019.PWM
- removed net POST-OPTO-DIODE: PC817.C, R1.2
- removed net RELAY-TO-MOTORCONTROLLER: RELAY2.P, TLE5205.VS
- removed net RELAY-TO-OPTO: D2.A, PC817.COL, RELAY1.2
- removed net SCL: MICRO.D3/SCL, SDA__SCL1.2, SDA__SCL2.2
- removed net SDA: MICRO.D2/SDA, SDA__SCL1.1, SDA__SCL2.1
- removed net TEMPERATURE1: MICRO.A1, TEMPERATURE1.2
- removed net TEMPERATURE2: MICRO.A5, TEMPERATURE2.2
- removed net VIN: MICRO.VIN, VIN-1.KL
- new net 3V3: SCREEN.6, U4.A, U4.RST, U4.VDD
- new net BLUE-NPN-BASE: R2.2, R5.2, T2.B
- new net BLUE-NPN-EMITTER: R6.2, T2.E
- new net GREEN-NPN-BASE: R10.2, R9.2, T4.B
- new net GREEN-NPN-EMITTER: R11.2, T4.E
- new net N$3: C5.2, U4.VOUT
- new net RED-NPN-BASE: R4.2, R7.2, T3.B
- new net RED-NPN-EMITTER: R8.2, T3.E
- new net SCREEN-BLUE: T2.C, U4.K-B
- new net SCREEN-BLUE-CONTROL: R2.1, SCREEN.5
- new net SCREEN-GREEN: T4.C, U4.K-G
- new net SCREEN-GREEN-CONTROL: R9.1, SCREEN.7
- new net SCREEN-RED: T3.C, U4.K-R
- new net SCREEN-RED-CONTROL: R4.1, SCREEN.9
- new net SCREEN-SCL: SCREEN.1, U4.SCL
- new net SCREEN-SDA: SCREEN.2, U4.SDA
- net GND: now also C5.1, R11.1, R5.1, R7.1, R8.1, SCREEN.10, SCREEN.3, SCREEN.4, SCREEN.8, U4.VSS; no longer 12V-2.KL, MICRO.GND, MICRO.GND1, PC817.EMIT, R1.1, R11.2, R3.2, TEMPERATURE1.1, TEMPERATURE2.1, TLE5205.GND, VIN-2.KL, VNH5019.GND1, VNH5019.GND2, VNH5019.GND3, VNH5019.GND4
- net N$21: now also C4.2, U4.C1+; no longer MICRO.D7
- net N$22: now also C4.1, U4.C1-; no longer MICRO.IO8
Other:
- note removed: "4 and 12 may not have PWM"
- moved on the sheet: R10, R11, R2, R6, R7, R8, R9

Commit message: MKII
Parts:
- R11, R6, R8: value 36 -> 33
Changed lines of the file:
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@@
 <?xml version="1.0" encoding="utf-8"?>
 <!DOCTYPE eagle SYSTEM "eagle.dtd">
-<eagle version="9.1.3">
+<eagle version="9.2.0">
 <drawing>
 <settings>
@@
 <part name="R2" library="resistor" library_urn="urn:adsk.eagle:library:348" deviceset="R-US_" device="0207/12" package3d_urn="urn:adsk.eagle:package:25938/1" value="1k"/>
 <part name="R5" library="resistor" library_urn="urn:adsk.eagle:library:348" deviceset="R-US_" device="0207/12" package3d_urn="urn:adsk.eagle:package:25938/1" value="47k"/>
-<part name="R6" library="resistor" library_urn="urn:adsk.eagle:library:348" deviceset="R-US_" device="0207/12" package3d_urn="urn:adsk.eagle:package:25938/1" value="36"/>
+<part name="R6" library="resistor" library_urn="urn:adsk.eagle:library:348" deviceset="R-US_" device="0207/12" package3d_urn="urn:adsk.eagle:package:25938/1" value="33"/>
 <part name="GND14" library="supply1" library_urn="urn:adsk.eagle:library:371" deviceset="GND" device=""/>
 <part name="T3" library="transistor" library_urn="urn:adsk.eagle:library:402" deviceset="2N2222" device="" package3d_urn="urn:adsk.eagle:package:28526/2"/>
 <part name="R4" library="resistor" library_urn="urn:adsk.eagle:library:348" deviceset="R-US_" device="0207/12" package3d_urn="urn:adsk.eagle:package:25938/1" value="1k"/>
 <part name="R7" library="resistor" library_urn="urn:adsk.eagle:library:348" deviceset="R-US_" device="0207/12" package3d_urn="urn:adsk.eagle:package:25938/1" value="47k"/>
-<part name="R8" library="resistor" library_urn="urn:adsk.eagle:library:348" deviceset="R-US_" device="0207/12" package3d_urn="urn:adsk.eagle:package:25938/1" value="36"/>
+<part name="R8" library="resistor" library_urn="urn:adsk.eagle:library:348" deviceset="R-US_" device="0207/12" package3d_urn="urn:adsk.eagle:package:25938/1" value="33"/>
 <part name="GND15" library="supply1" library_urn="urn:adsk.eagle:library:371" deviceset="GND" device=""/>
 <part name="T4" library="transistor" library_urn="urn:adsk.eagle:library:402" deviceset="2N2222" device="" package3d_urn="urn:adsk.eagle:package:28526/2"/>
 <part name="R9" library="resistor" library_urn="urn:adsk.eagle:library:348" deviceset="R-US_" device="0207/12" package3d_urn="urn:adsk.eagle:package:25938/1" value="1k"/>
 <part name="R10" library="resistor" library_urn="urn:adsk.eagle:library:348" deviceset="R-US_" device="0207/12" package3d_urn="urn:adsk.eagle:package:25938/1" value="47k"/>
-<part name="R11" library="resistor" library_urn="urn:adsk.eagle:library:348" deviceset="R-US_" device="0207/12" package3d_urn="urn:adsk.eagle:package:25938/1" value="36"/>
+<part name="R11" library="resistor" library_urn="urn:adsk.eagle:library:348" deviceset="R-US_" device="0207/12" package3d_urn="urn:adsk.eagle:package:25938/1" value="33"/>
 <part name="GND16" library="supply1" library_urn="urn:adsk.eagle:library:371" deviceset="GND" device=""/>
 <part name="U4" library="GEMS" deviceset="NHD‐C0220" device=""/>
@@
 </plain>
 <instances>
-<instance part="SCREEN" gate="G$1" x="138.43" y="15.24"/>
-<instance part="GND12" gate="1" x="146.05" y="7.62"/>
-<instance part="GND13" gate="1" x="168.91" y="15.24"/>
-<instance part="T2" gate="G$1" x="186.69" y="48.26"/>
-<instance part="R2" gate="G$1" x="168.91" y="48.26"/>
-<instance part="R5" gate="G$1" x="179.07" y="35.56" rot="R90"/>
-<instance part="R6" gate="G$1" x="189.23" y="35.56" rot="R90"/>
-<instance part="GND14" gate="1" x="189.23" y="25.4"/>
-<instance part="T3" gate="G$1" x="278.13" y="48.26"/>
-<instance part="R4" gate="G$1" x="260.35" y="48.26"/>
-<instance part="R7" gate="G$1" x="270.51" y="35.56" rot="R90"/>
-<instance part="R8" gate="G$1" x="280.67" y="35.56" rot="R90"/>
-<instance part="GND15" gate="1" x="280.67" y="25.4"/>
-<instance part="T4" gate="G$1" x="372.11" y="48.26"/>
-<instance part="R9" gate="G$1" x="354.33" y="48.26"/>
-<instance part="R10" gate="G$1" x="364.49" y="35.56" rot="R90"/>
-<instance part="R11" gate="G$1" x="374.65" y="35.56" rot="R90"/>
-<instance part="GND16" gate="1" x="374.65" y="25.4"/>
-<instance part="U4" gate="G$1" x="62.23" y="48.26"/>
-<instance part="C4" gate="G$1" x="92.71" y="40.64"/>
-<instance part="C5" gate="G$1" x="82.55" y="15.24" rot="R90"/>
-<instance part="GND18" gate="1" x="80.01" y="7.62"/>
+<instance part="SCREEN" gate="G$1" x="138.43" y="15.24">
+<attribute name="VALUE" x="134.62" y="5.334" size="1.778" layer="96" font="vector"/>
+<attribute name="NAME" x="134.62" y="23.368" size="1.778" layer="95" font="vector"/>
+</instance>
+<instance part="GND12" gate="1" x="146.05" y="7.62">
+<attribute name="VALUE" x="143.51" y="5.08" size="1.778" layer="96"/>
+</instance>
+<instance part="GND13" gate="1" x="168.91" y="15.24">
+<attribute name="VALUE" x="166.37" y="12.7" size="1.778" layer="96"/>
+</instance>
+<instance part="T2" gate="G$1" x="186.69" y="48.26">
+<attribute name="NAME" x="176.53" y="55.88" size="1.778" layer="95"/>
+<attribute name="VALUE" x="176.53" y="53.34" size="1.778" layer="96"/>
+</instance>
+<instance part="R2" gate="G$1" x="168.91" y="48.26">
+<attribute name="NAME" x="165.1" y="49.7586" size="1.778" layer="95"/>
+<attribute name="VALUE" x="165.1" y="44.958" size="1.778" layer="96"/>
+</instance>
+<instance part="R5" gate="G$1" x="179.07" y="35.56" rot="R90">
+<attribute name="NAME" x="177.5714" y="31.75" size="1.778" layer="95" rot="R90"/>
+<attribute name="VALUE" x="182.372" y="31.75" size="1.778" layer="96" rot="R90"/>
+</instance>
+<instance part="R6" gate="G$1" x="189.23" y="35.56" rot="R90">
+<attribute name="NAME" x="187.7314" y="31.75" size="1.778" layer="95" rot="R90"/>
+<attribute name="VALUE" x="192.532" y="31.75" size="1.778" layer="96" rot="R90"/>
+</instance>
+<instance part="GND14" gate="1" x="189.23" y="25.4">
+<attribute name="VALUE" x="186.69" y="22.86" size="1.778" layer="96"/>
+</instance>
+<instance part="T3" gate="G$1" x="278.13" y="48.26">
+<attribute name="NAME" x="267.97" y="55.88" size="1.778" layer="95"/>
+<attribute name="VALUE" x="267.97" y="53.34" size="1.778" layer="96"/>
+</instance>
+<instance part="R4" gate="G$1" x="260.35" y="48.26">
+<attribute name="NAME" x="256.54" y="49.7586" size="1.778" layer="95"/>
+<attribute name="VALUE" x="256.54" y="44.958" size="1.778" layer="96"/>
+</instance>
+<instance part="R7" gate="G$1" x="270.51" y="35.56" rot="R90">
+<attribute name="NAME" x="269.0114" y="31.75" size="1.778" layer="95" rot="R90"/>
+<attribute name="VALUE" x="273.812" y="31.75" size="1.778" layer="96" rot="R90"/>
+</instance>
+<instance part="R8" gate="G$1" x="280.67" y="35.56" rot="R90">
+<attribute name="NAME" x="279.1714" y="31.75" size="1.778" layer="95" rot="R90"/>
+<attribute name="VALUE" x="283.972" y="31.75" size="1.778" layer="96" rot="R90"/>
+</instance>
+<instance part="GND15" gate="1" x="280.67" y="25.4">
+<attribute name="VALUE" x="278.13" y="22.86" size="1.778" layer="96"/>
+</instance>
+<instance part="T4" gate="G$1" x="372.11" y="48.26">
+<attribute name="NAME" x="361.95" y="55.88" size="1.778" layer="95"/>
+<attribute name="VALUE" x="361.95" y="53.34" size="1.778" layer="96"/>
+</instance>
+<instance part="R9" gate="G$1" x="354.33" y="48.26">
+<attribute name="NAME" x="350.52" y="49.7586" size="1.778" layer="95"/>
+<attribute name="VALUE" x="350.52" y="44.958" size="1.778" layer="96"/>
+</instance>
+<instance part="R10" gate="G$1" x="364.49" y="35.56" rot="R90">
+<attribute name="NAME" x="362.9914" y="31.75" size="1.778" layer="95" rot="R90"/>
+<attribute name="VALUE" x="367.792" y="31.75" size="1.778" layer="96" rot="R90"/>
+</instance>
+<instance part="R11" gate="G$1" x="374.65" y="35.56" rot="R90">
+<attribute name="NAME" x="373.1514" y="31.75" size="1.778" layer="95" rot="R90"/>
+<attribute name="VALUE" x="377.952" y="31.75" size="1.778" layer="96" rot="R90"/>
+</instance>
+<instance part="GND16" gate="1" x="374.65" y="25.4">
+<attribute name="VALUE" x="372.11" y="22.86" size="1.778" layer="96"/>
+</instance>
+<instance part="U4" gate="G$1" x="62.23" y="48.26">
+<attribute name="NAME" x="62.23" y="63.754" size="1.27" layer="95"/>
+<attribute name="VALUE" x="62.23" y="61.722" size="1.27" layer="96"/>
+</instance>
+<instance part="C4" gate="G$1" x="92.71" y="40.64">
+<attribute name="NAME" x="94.234" y="41.021" size="1.778" layer="95"/>
+<attribute name="VALUE" x="94.234" y="35.941" size="1.778" layer="96"/>
+</instance>
+<instance part="C5" gate="G$1" x="82.55" y="15.24" rot="R90">
+<attribute name="NAME" x="82.169" y="16.764" size="1.778" layer="95" rot="R90"/>
+<attribute name="VALUE" x="87.249" y="16.764" size="1.778" layer="96" rot="R90"/>
+</instance>
+<instance part="GND18" gate="1" x="80.01" y="7.62">
+<attribute name="VALUE" x="77.47" y="5.08" size="1.778" layer="96"/>
+</instance>
 </instances>
 <busses>
